Commit message: 20250928

File: description/ros2_control/carlikebot.ros2_control.xacro (robot description, xacro)
@@ -1,5 +1,5 @@
 <?xml version="1.0"?>
 <robot xmlns:xacro="http://www.ros.org/wiki/xacro">
-  <xacro:macro name="carlikebot_ros2_control" params="name prefix">
+  <xacro:macro name="carlikebot_ros2_control" params="name">
     <ros2_control name="${name}" type="system">
       <hardware>
@@ -8,9 +8,9 @@
         <param name="example_param_hw_stop_duration_sec">3.0</param>
       </hardware>
-      <joint name="${prefix}virtual_front_wheel_joint">
+      <joint name="virtual_front_wheel_joint">
         <command_interface name="position"/>
         <state_interface name="position"/>
       </joint>
-      <joint name="${prefix}virtual_rear_wheel_joint">
+      <joint name="virtual_rear_wheel_joint">
         <command_interface name="velocity"/>
         <state_interface name="velocity"/>

File: description/urdf/carlikebot.urdf.xacro (robot description, xacro)
@@ -2,12 +2,8 @@
 <!-- 4 Wheel Robot with front steering and rear drive -->
 <robot xmlns:xacro="http://www.ros.org/wiki/xacro" name="carlikebot_robot">
-  <xacro:arg name="prefix" default="" />
-  <xacro:include filename="$(find ros2_control_demo_description)/carlikebot/urdf/carlikebot_description.urdf.xacro" />
-  <!-- Import Rviz colors -->
-  <xacro:include filename="$(find ros2_control_demo_description)/carlikebot/urdf/carlikebot.materials.xacro" />
-  <!-- Import carlikebot ros2_control description -->
-  <xacro:include filename="$(find ros2_control_demo_example_11)/ros2_control/carlikebot.ros2_control.xacro" />
-  <xacro:carlikebot prefix="$(arg prefix)" />
-  <xacro:carlikebot_ros2_control
-    name="CarlikeBot" prefix="$(arg prefix)" />
+  <xacro:include filename="$(find robot_controller2_ackm)/description/urdf/tt02.xacro" />
+  <xacro:include
+    filename="$(find robot_controller2_ackm)/description/ros2_control/carlikebot.ros2_control.xacro" />
+  <xacro:tt02_body />
+  <xacro:carlikebot_ros2_control name="CarlikeBot" />
 </robot>

Commit message: 20250928

File: description/ros2_control/carlikebot.ros2_control.xacro (robot description, xacro)
@@ -4,5 +4,5 @@
     <ros2_control name="${name}" type="system">
       <hardware>
-        <plugin>test_control_ackm/CarlikeBotSystemHardware</plugin>
+        <plugin>robot_controller2_ackm/CarlikeBotSystemHardware</plugin>
         <param name="example_param_hw_start_duration_sec">0</param>
         <param name="example_param_hw_stop_duration_sec">3.0</param>

File: description/urdf/carlikebot.urdf.xacro (robot description, xacro)
@@ -2,7 +2,7 @@
 <!-- 4 Wheel Robot with front steering and rear drive -->
 <robot xmlns:xacro="http://www.ros.org/wiki/xacro" name="carlikebot_robot">
-  <xacro:include filename="$(find robot_controller2_ackm)/description/urdf/tt02.xacro" />
+  <xacro:include filename="$(find robot_controller2_ackm)/urdf/tt02.xacro" />
   <xacro:include
-    filename="$(find robot_controller2_ackm)/description/ros2_control/carlikebot.ros2_control.xacro" />
+    filename="$(find robot_controller2_ackm)/ros2_control/carlikebot.ros2_control.xacro" />
   <xacro:tt02_body />
   <xacro:carlikebot_ros2_control name="CarlikeBot" />

File: description/urdf/tt02.xacro (robot description, xacro)
@@ -2,5 +2,5 @@
 <!-- 4 wheel car with front steering and rear drive based on Tamiya TT02 -->
 <robot xmlns:xacro="http://www.ros.org/wiki/xacro">
-  <xacro:macro name="tt02_body" params="name prefix">
+  <xacro:macro name="tt02_body">
     <!--==================================================
       ===== Define robot constants                 =====
@@ -98,5 +98,5 @@
       <parent link="base_link" />
       <child link="base_body" />
-      <origin xyz="0.0 0.0 0.0}" rpy="0 0 0" />
+      <origin xyz="0.0 0.0 0.0" rpy="0 0 0" />
     </joint>
     <!-- Robot Footprint -->
