Commit message: 20251004

File: description/urdf/tt02.xacro (robot description, xacro)
@@ -154,5 +154,5 @@
         <limit effort="100.0" velocity="100.0" />
         <dynamics damping="0.2" />
-        <mimic joint="${prefix}virtual_rear_wheel_joint" multiplier="1.0" offset="0.0" />
+        <mimic joint="virtual_rear_wheel_joint" multiplier="1.0" offset="0.0" />
       </joint>
       <gazebo reference="${prefix}_joint">

Commit message: 20251012

File: description/urdf/tt02.xacro (robot description, xacro)
@@ -22,7 +22,7 @@
     <!-- <xacro:property name="caster_base_height"
     value="${wheel_radius+wheel_zoff-(base_height/2)-(caster_radius*2)}" /> -->
-    <!-- <xacro:property name="lidar_xoff" value="0.05" /> -->
-    <!-- <xacro:property name="lidar_height" value="0.06" /> -->
-    <!-- <xacro:property name="lidar_radius" value="0.035" /> -->
+    <xacro:property name="lidar_xoff" value="0.05" />
+    <xacro:property name="lidar_height" value="0.06" />
+    <xacro:property name="lidar_radius" value="0.035" />
     <!-- <xacro:property name="battery_width" value="${base_width}" /> -->
     <!-- <xacro:property name="battery_length" value="0.09" /> -->
@@ -44,5 +44,5 @@
     <!-- <xacro:property name="caster_mass" value="0.05" /> -->
     <!-- <xacro:property name="battery_mass" value="0.107" /> -->
-    <!-- <xacro:property name="lidar_mass" value="0.17" /> -->
+    <xacro:property name="lidar_mass" value="0.17" />
     <!-- <xacro:property name="imu_mass" value="0.0544" /> -->
     <!-- <xacro:property name="raspi_mass" value="0.047" /> -->

Commit message: 20251012

File: description/urdf/tt02.xacro (robot description, xacro)
@@ -22,7 +22,7 @@
     <!-- <xacro:property name="caster_base_height"
     value="${wheel_radius+wheel_zoff-(base_height/2)-(caster_radius*2)}" /> -->
-    <xacro:property name="lidar_xoff" value="0.05" />
-    <xacro:property name="lidar_height" value="0.06" />
-    <xacro:property name="lidar_radius" value="0.035" />
+    <!-- <xacro:property name="lidar_xoff" value="0.05" /> -->
+    <!-- <xacro:property name="lidar_height" value="0.06" /> -->
+    <!-- <xacro:property name="lidar_radius" value="0.035" /> -->
     <!-- <xacro:property name="battery_width" value="${base_width}" /> -->
     <!-- <xacro:property name="battery_length" value="0.09" /> -->
@@ -44,5 +44,5 @@
     <!-- <xacro:property name="caster_mass" value="0.05" /> -->
     <!-- <xacro:property name="battery_mass" value="0.107" /> -->
-    <xacro:property name="lidar_mass" value="0.17" />
+    <!-- <xacro:property name="lidar_mass" value="0.17" /> -->
     <!-- <xacro:property name="imu_mass" value="0.0544" /> -->
     <!-- <xacro:property name="raspi_mass" value="0.047" /> -->
@@ -225,6 +225,5 @@
     <xacro:front_wheel prefix="drivewheel_fronr_right" y_reflect="-1" />
     <!-- Import carlikebot ros2_control description -->
-    <!-- <xacro:include filename="$(find
-  ros2_control_demo_example_11)/ros2_control/carlikebot.ros2_control.xacro" /> -->
+    <!-- <xacro:include filename="$(find  ros2_control_demo_example_11)/ros2_control/carlikebot.ros2_control.xacro" /> -->
     <!-- <xacro:carlikebot prefix="$(arg prefix)" /> -->
     <!-- <xacro:carlikebot_ros2_control name="CarlikeBot" prefix="$(arg prefix)" /> -->

Commit message: 20251012

File: description/urdf/tt02.xacro (robot description, xacro)
@@ -22,7 +22,7 @@
     <!-- <xacro:property name="caster_base_height"
     value="${wheel_radius+wheel_zoff-(base_height/2)-(caster_radius*2)}" /> -->
-    <!-- <xacro:property name="lidar_xoff" value="0.05" /> -->
-    <!-- <xacro:property name="lidar_height" value="0.06" /> -->
-    <!-- <xacro:property name="lidar_radius" value="0.035" /> -->
+    <xacro:property name="lidar_xoff" value="0.05" />
+    <xacro:property name="lidar_height" value="0.045" />
+    <xacro:property name="lidar_radius" value="0.035" />
     <!-- <xacro:property name="battery_width" value="${base_width}" /> -->
     <!-- <xacro:property name="battery_length" value="0.09" /> -->
@@ -44,5 +44,5 @@
     <!-- <xacro:property name="caster_mass" value="0.05" /> -->
     <!-- <xacro:property name="battery_mass" value="0.107" /> -->
-    <!-- <xacro:property name="lidar_mass" value="0.17" /> -->
+    <xacro:property name="lidar_mass" value="0.17" />
     <!-- <xacro:property name="imu_mass" value="0.0544" /> -->
     <!-- <xacro:property name="raspi_mass" value="0.047" /> -->
@@ -224,6 +224,64 @@
     <xacro:front_wheel prefix="drivewheel_front_left" y_reflect="1" />
     <xacro:front_wheel prefix="drivewheel_fronr_right" y_reflect="-1" />
+    <!-- Laidar -->
+    <link name="laser">
+      <inertial>
+        <origin xyz="0 0 0" rpy="0 0 0" />
+        <mass value="${lidar_mass}" />
+        <inertia ixx="0.001" ixy="0" ixz="0" iyy="0.001" iyz="0" izz="0.001" />
+      </inertial>
+      <collision name="laser_collision">
+        <origin xyz="0 0 0" rpy="0 0 0" />
+        <geometry>
+          <cylinder radius="${lidar_radius}" length="${lidar_height}" />
+        </geometry>
+      </collision>
+      <visual name="laser_visual">
+        <origin xyz="0 0 0" rpy="0 0 0" />
+        <geometry>
+          <cylinder radius="${lidar_radius}" length="${lidar_height}" />
+        </geometry>
+        <material name="Cyan">
+          <color rgba="0 1.0 1.0 1.0" />
+        </material>
+      </visual>
+    </link>
+    <!-- <gazebo reference="laser">
+      <sensor name="rplidar" type="gpu_lidar">
+        <always_on>true</always_on>
+        <visualize>true</visualize>
+        <update_rate>5</update_rate>
+        <topic>scan</topic>
+        <ignition_frame_id>laser</ignition_frame_id>
+        <lidar>
+          <scan>
+            <horizontal>
+              <samples>360</samples>
+              <resolution>1.0</resolution>
+              <min_angle>0.0</min_angle>
+              <max_angle>6.28</max_angle>
+            </horizontal>
+          </scan>
+          <range>
+            <min>0.15</min>
+            <max>12</max>
+            <resolution>0.0005</resolution>
+          </range>
+          <noise>
+            <type>gaussian</type>
+            <mean>0.0</mean>
+            <stddev>0.01</stddev>
+          </noise>
+        </lidar>
+      </sensor>
+    </gazebo> -->
+    <joint name="lidar_joint" type="fixed">
+      <parent link="base_link" />
+      <child link="laser" />
+      <origin xyz="${lidar_xoff} 0.0 ${base_height/2+lidar_height/2}" rpy="0 0 0" />
+    </joint>
     <!-- Import carlikebot ros2_control description -->
-    <!-- <xacro:include filename="$(find  ros2_control_demo_example_11)/ros2_control/carlikebot.ros2_control.xacro" /> -->
+    <!-- <xacro:include filename="$(find
+    ros2_control_demo_example_11)/ros2_control/carlikebot.ros2_control.xacro" /> -->
     <!-- <xacro:carlikebot prefix="$(arg prefix)" /> -->
     <!-- <xacro:carlikebot_ros2_control name="CarlikeBot" prefix="$(arg prefix)" /> -->

Commit message: 20251013

File: description/urdf/tt02.xacro (robot description, xacro)
@@ -28,7 +28,8 @@
     <!-- <xacro:property name="battery_length" value="0.09" /> -->
     <!-- <xacro:property name="battery_height" value="0.025" /> -->
-    <!-- <xacro:property name="imu_width" value="0.06" /> -->
-    <!-- <xacro:property name="imu_length" value="0.045" /> -->
-    <!-- <xacro:property name="imu_height" value="0.01" /> -->
+    <xacro:property name="imu_xoff" value="0.02" />
+    <xacro:property name="imu_width" value="0.06" />
+    <xacro:property name="imu_length" value="0.045" />
+    <xacro:property name="imu_height" value="0.01" />
     <!-- <xacro:property name="raspi_xoff" value="0.067" /> -->
     <!-- <xacro:property name="raspi_width" value="0.085" /> -->
@@ -45,5 +46,5 @@
     <!-- <xacro:property name="battery_mass" value="0.107" /> -->
     <xacro:property name="lidar_mass" value="0.17" />
-    <!-- <xacro:property name="imu_mass" value="0.0544" /> -->
+    <xacro:property name="imu_mass" value="0.0544" />
     <!-- <xacro:property name="raspi_mass" value="0.047" /> -->
     <!-- <xacro:property name="camera_mass" value="0.047" /> -->
@@ -281,4 +282,87 @@
       <origin xyz="${lidar_xoff} 0.0 ${base_height/2+lidar_height/2}" rpy="0 0 0" />
     </joint>
+    <!-- IMU -->
+    <link name="imu_link">
+      <visual>
+        <geometry>
+          <box size="${imu_length} ${imu_width} ${imu_height}" />
+        </geometry>
+        <material name="Cyan">
+          <color rgba="0 1.0 1.0 1.0" />
+        </material>
+      </visual>
+      <collision>
+        <geometry>
+          <box size="${imu_length} ${imu_width} ${imu_height}" />
+        </geometry>
+      </collision>
+      <xacro:box_inertia m="${imu_mass}" w="${imu_width}" d="${imu_length}" h="${imu_height}" />
+    </link>
+    <!-- <gazebo reference="imu_link">
+      <sensor name="yahboom" type="imu">
+        <always_on>true</always_on>
+        <update_rate>100</update_rate>
+        <topic>imu/data_raw</topic>
+        <imu>
+          <angular_velocity>
+            <x>
+              <noise type="gaussian">
+                <mean>0.0</mean>
+                <stddev>2e-4</stddev>
+                <bias_mean>0.0000075</bias_mean>
+                <bias_stddev>0.0000008</bias_stddev>
+              </noise>
+            </x>
+            <y>
+              <noise type="gaussian">
+                <mean>0.0</mean>
+                <stddev>2e-4</stddev>
+                <bias_mean>0.0000075</bias_mean>
+                <bias_stddev>0.0000008</bias_stddev>
+              </noise>
+            </y>
+            <z>
+              <noise type="gaussian">
+                <mean>0.0</mean>
+                <stddev>2e-4</stddev>
+                <bias_mean>0.0000075</bias_mean>
+                <bias_stddev>0.0000008</bias_stddev>
+              </noise>
+            </z>
+          </angular_velocity>
+          <linear_acceleration>
+            <x>
+              <noise type="gaussian">
+                <mean>0.0</mean>
+                <stddev>1.7e-2</stddev>
+                <bias_mean>0.1</bias_mean>
+                <bias_stddev>0.001</bias_stddev>
+              </noise>
+            </x>
+            <y>
+              <noise type="gaussian">
+                <mean>0.0</mean>
+                <stddev>1.7e-2</stddev>
+                <bias_mean>0.1</bias_mean>
+                <bias_stddev>0.001</bias_stddev>
+              </noise>
+            </y>
+            <z>
+              <noise type="gaussian">
+                <mean>0.0</mean>
+                <stddev>1.7e-2</stddev>
+                <bias_mean>0.1</bias_mean>
+                <bias_stddev>0.001</bias_stddev>
+              </noise>
+            </z>
+          </linear_acceleration>
+        </imu>
+      </sensor>
+    </gazebo> -->
+    <joint name="imu_joint" type="fixed">
+      <parent link="base_link" />
+      <child link="imu_link" />
+      <origin xyz="$-{imu_xoff} 0.0 ${base_height/2+imu_height/2}" />
+    </joint>
     <!-- Import carlikebot ros2_control description -->
     <!-- <xacro:include filename="$(find

Commit message: 20251018

File: description/urdf/tt02.xacro (robot description, xacro)
@@ -363,5 +363,5 @@
       <parent link="base_link" />
       <child link="imu_link" />
-      <origin xyz="$-{imu_xoff} 0.0 ${base_height/2+imu_height/2}" />
+      <origin xyz="${-imu_xoff} 0.0 ${base_height/2+imu_height/2}" />
     </joint>
     <!-- Import carlikebot ros2_control description -->
